File: IFT-S3.kicad_sch (KiCad schematic)
At the start: 17 parts, among them J1 Conn_01x04_Socket, J2 Conn_01x01_Pin, J3 Conn_01x02_Pin, J6 Conn_01x02_Pin, J7 Conn_01x02, Q1 Q_Photo_NPN, Q2 Q_NMOS_GSD, Q3 IRFZ44N, U1 XIAO-ESP32-S3-DIP

Commit message: Clean up and OLED 3D model added
Connections:
- net Tr_DRAIN: no longer names the net of J3.1 (Pin_1), J6.1 (Pin_1), Q2.3 (D), Q3.2 (D)
Other:
- note added: "Keyboard"
- note added: "Light sensor (optional)"
- note added: "MOSFET (optional)"
- note added: "Neopixel RGB LED (optional)"
- note added: "Power switch and battery connector (optional)"
- note added: "Solder only one of the two transistors !"
- note added: "Xiao ESP S3 connector"
- note removed: "Light sensor"
- note removed: "MOSFET"
- note removed: "Neopixel RGB LED"
- note removed: "Solder only one of the transistor"
- company: (none) -> IFT
- title: (none) -> IFT-S3
- moved on the sheet: J3, J6, Q1, Q2, Q3, R11, R14
