File: IFT-S3.kicad_sch (KiCad schematic)
At the start: 17 parts, among them J1 Conn_01x04_Socket, J2 Conn_01x01_Pin, J3 Conn_01x02_Pin, J6 Conn_01x02_Pin, J7 Conn_01x02, Q1 Q_Photo_NPN, Q2 Q_NMOS_GSD, Q3 IRFZ44N, U1 XIAO-ESP32-S3-DIP

Commit message: Postion of Xiao battery connector fixed
Parts:
- Q3: value IRFZ44N -> IRLZ44N
Changed lines of the file:
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@@
 		)
 		(instances
-			(project ""
+			(project "IFT-S3"
 				(path "/9106ad3b-5dea-4727-91ce-50cc3919a94c"
 					(reference "J2")
@@
 			)
 		)
-		(property "Value" "IRFZ44N"
+		(property "Value" "IRLZ44N"
 			(at 247.65 149.8599 0)
 			(effects
@@
 			)
 		)
-		(property "Datasheet" "http://www.infineon.com/dgdl/irf4905.pdf?fileId=5546d462533600a4015355e32165197c"
+		(property "Datasheet" ""
 			(at 246.38 152.4 0)
 			(effects
@@
 			)
 		)
-		(property "Description" "-74A Id, -55V Vds, Single P-Channel HEXFET Power MOSFET, 20mOhm Ron, TO-220AB"
+		(property "Description" ""
 			(at 241.3 148.59 0)
 			(effects
@@
 		)
 		(instances
-			(project ""
+			(project "IFT-S3"
 				(path "/9106ad3b-5dea-4727-91ce-50cc3919a94c"
 					(reference "Q3")
@@
 		)
 		(instances
-			(project ""
+			(project "IFT-S3"
 				(path "/9106ad3b-5dea-4727-91ce-50cc3919a94c"
 					(reference "U1")

Commit message: Final version (2026) sent to production
Parts:
- removed J6: Conn_01x02_Pin, Motors:Vybronics_VZ30C1T8219732L, symbol Connector:Conn_01x02_Pin
- removed Q1: Q_Photo_NPN, Local footprints:SFH3710, symbol Device:Q_Photo_NPN
- removed R11: 1M, Resistor_SMD:R_0805_2012Metric_Pad1.20x1.40mm_HandSolder, symbol Device:R
- added J4: Conn_01x02_Pin, Connector_PinHeader_2.54mm:PinHeader_1x02_P2.54mm_Vertical, symbol Connector:Conn_01x02_Pin
- added J5, J6: Conn_01x01_Pin, Connector_PinHeader_2.54mm:PinHeader_1x01_P2.54mm_Vertical, symbol Connector:Conn_01x01_Pin
- added Q4: Q_NMOS_GSD, Package_TO_SOT_SMD:SOT-23-3, symbol Device:Q_NMOS_GSD
- added Q5: IRLZ44N, Package_TO_SOT_THT:TO-220-3_Vertical, symbol Transistor_FET:IRF4905
- added R15: 10K, Resistor_SMD:R_0805_2012Metric_Pad1.20x1.40mm_HandSolder, symbol Device:R
Connections:
- net +3.3V: now also J4.2 (Pin_2)
- net GND: now also Q4.2 (S), Q5.3 (S), R15.2
- net RGB_OUT: now also J5.1 (Pin_1)
- net Tr_GATE: now also Q4.1 (G), Q5.1 (G), R15.1; no longer Q2.1 (G), Q3.1 (G), R14.1
- net drain2: now reaches J3.1 (Pin_1), Q2.3 (D), Q3.2 (D)
- net at U1.14 (VBUS): now also J6.1 (Pin_1)
- net Photo_Tr renamed Tr_GATE2
- net Tr_GATE2: now also Q2.1 (G), Q3.1 (G), R14.1
- new net drain: J4.1 (Pin_1), Q4.3 (D), Q5.2 (D)
- no-connect marks 1 -> 0
Other:
- note added: "MOSFET (left)"
- note added: "MOSFET (right)"
- note removed: "Light sensor (optional)"
- note removed: "MOSFET (optional)"
- moved on the sheet: J3
