File: IFT-S3.kicad_pcb (KiCad board)
At the start: 2 copper layers, 54 x 85.6 mm, 38 parts, among them J1 Conn_01x04_Socket, J2 Conn_01x01_Pin, J3 Conn_01x02_Pin, J6 Conn_01x02_Pin, J7 Conn_01x02, Q1 Q_Photo_NPN, Q2 Q_NMOS_GSD, Q3 IRFZ44N, SW2 PTS526_SK15_SMTR2_LFS, SW3 PTS526_SK15_SMTR2_LFS, SW4 PTS526_SK15_SMTR2_LFS, SW5 PTS526_SK15_SMTR2_LFS, SW6 PTS526_SK15_SMTR2_LFS, SW7 PTS526_SK15_SMTR2_LFS, SW8 PTS526_SK15_SMTR2_LFS, SW9 PTS526_SK15_SMTR2_LFS, U1 XIAO-ESP32-S3-DIP

Commit message: Postion of Xiao battery connector fixed
Parts:
- removed the REF** at (128.0, 130.6)
- Q3: value IRFZ44N -> IRLZ44N
- moved J2 8.63 mm to (155.4, 126.1)
- moved D1 0.75 mm to (142.4, 100.3)
Connections:
- net Tr_DRAIN renamed Net-(J3-Pin_1)
Routing:
- net +BATT_after_switch: track 71.4 -> 75.0 mm
- net Photo_Tr: track 98.3 -> 101.2 mm
- net Net-(D1-A): track 8.55 -> 9.16 mm

Commit message: Final version (2026) sent to production
Parts:
- removed Q1: Q_Photo_NPN, Local footprints:SFH3710
- removed R11: 1M, Resistor_SMD:R_0805_2012Metric_Pad1.20x1.40mm_HandSolder
- removed SW9: PTS526_SK15_SMTR2_LFS, footprints:PTS526SK15SMTR2LFS
- added J4: Conn_01x02_Pin, Connector_PinHeader_2.54mm:PinHeader_1x02_P2.54mm_Vertical, F.Cu at (175.6, 84.8)
- added J5: Conn_01x01_Pin, Connector_PinHeader_2.54mm:PinHeader_1x01_P2.54mm_Vertical, F.Cu at (174.0, 61.1)
- added Q4: Q_NMOS_GSD, Package_TO_SOT_SMD:SOT-23-3, F.Cu at (172.2, 74.1)
- added Q5: IRLZ44N, Package_TO_SOT_THT:TO-220-3_Vertical, F.Cu at (169.6, 80.4)
- added R15: 10K, Resistor_SMD:R_0805_2012Metric_Pad1.20x1.40mm_HandSolder, F.Cu at (175.5, 91.4)
- added REF**: OSHW-Logo_11.4x12mm_Mask, footprints:OSHW-Logo_11.4x12mm_Mask, F.Cu at (152.0, 94.7)
- added REF**: Fiducial_0.5mm_Mask1.5mm, Fiducial:Fiducial_0.5mm_Mask1.5mm, F.Cu at (128.0, 60.5)
- added SW1: PTS526_SK15_SMTR2_LFS, footprints:PTS526SK15SMTR2LFS, F.Cu at (136.2, 99.8)
- J6: value Conn_01x02_Pin -> Conn_01x01_Pin; footprint Motors:Vybronics_VZ30C1T8219732L -> Connector_PinHeader_2.54mm:PinHeader_1x01_P2.54mm_Vertical
- REF**: moved to B.Cu
- moved J6 67.1 mm to (128.0, 129.4), turned to 0 degrees
- moved REF** 59.5 mm to (172.7, 128.2), turned to -90 degrees
- moved REF** 49.5 mm to (172.7, 120.7), turned to -90 degrees
- moved J3 46.3 mm to (126.6, 84.3), turned to 0 degrees
- moved Q2 45.2 mm to (130.0, 73.6)
- moved Q3 44.5 mm to (127.3, 80.2)
- moved SW4 44.0 mm to (128.2, 107.8), turned to -90 degrees
- moved R14 43.7 mm to (126.6, 90.8), turned to -90 degrees
- moved REF** 39.8 mm to (172.7, 113.2), turned to -90 degrees
- moved SW8 34.1 mm to (166.2, 132.0), turned to 90 degrees
- moved SW6 34.0 mm to (160.0, 107.8), turned to -155 degrees
- moved SW3 28.1 mm to (172.0, 103.5), turned to -155 degrees
- moved SW5 25.5 mm to (136.2, 132.0), turned to -90 degrees
- moved SW7 25.1 mm to (136.2, 115.8), turned to 0 degrees
- moved REF** 19.4 mm to (151.3, 77.0), turned to 180 degrees
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Connections:
- J3 pad 1: Net-(J3-Pin_1) -> /drain2
- J6 pad 1: Net-(J3-Pin_1) -> Net-(J6-Pin_1)
- Q2 pad 1: Tr_GATE -> Tr_GATE2
- Q2 pad 3: Net-(J3-Pin_1) -> /drain2
- Q3 pad 1: Tr_GATE -> Tr_GATE2
- Q3 pad 2: Net-(J3-Pin_1) -> /drain2
- R14 pad 1: Tr_GATE -> Tr_GATE2
- SW2 pad 1: O_1 -> O_2
- SW2 pad 2: O_1 -> Net-(D6-A)
- SW3 pad 1: O_2 -> O_3
- SW3 pad 2: O_2 -> Net-(D9-A)
- SW4 pad 1: O_3 -> O_1
- SW4 pad 2: O_3 -> Net-(D2-A)
- SW5 pad 1: O_1 -> O_2
- SW5 pad 2: O_1 -> Net-(D7-A)
- SW6 pad 1: O_2 -> O_3
- SW6 pad 2: O_2 -> Net-(D10-A)
- SW7 pad 1: O_3 -> O_1
- SW7 pad 2: O_3 -> Net-(D3-A)
- SW8 pad 1: O_1 -> O_2
- SW8 pad 2: O_1 -> Net-(D8-A)
- U1 pad 14: unconnected-(U1-VBUS-Pad14) -> Net-(J6-Pin_1)
- U1 pad 3: Photo_Tr -> Tr_GATE2
Routing:
- net Photo_Tr: track 101.2 -> 0.00 mm
- net Tr_GATE2: track 0.00 -> 81.3 mm, vias 0 -> 2
- net +3.3V: track 175.4 -> 149.4 mm, vias 2 -> 1
- net Tr_GATE: track 51.7 -> 77.1 mm, vias 0 -> 1
- net Net-(J6-Pin_1): track 0.00 -> 20.7 mm
- net O_2: track 67.4 -> 85.8 mm
- net /drain: track 0.00 -> 13.3 mm
- net /drain2: track 0.00 -> 13.2 mm
- net Net-(J3-Pin_1): track 13.0 -> 0.00 mm
- net /RGB_OUT: track 5.64 -> 17.3 mm
- net I_1: track 30.9 -> 40.8 mm
- net O_3: track 18.8 -> 27.9 mm
- net Net-(D2-A): track 2.48 -> 11.4 mm
- net +BATT: track 22.3 -> 13.6 mm
- net Net-(D10-A): track 6.40 -> 14.5 mm
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Other:
- board text added: "+3V3"
- board text added: "+5V (USB)"
- board text added: "+Batt"
- board text added: "Battery"
- board text added: "Createch 2026/2027"
- board text added: "GND"
- board text added: "RGB Out"
- board text added: "https://github.com/Acathla-fr/IFT-S3"
- board text removed: "Ambiant Light Sensor"
