File: keyboard_matrix.kicad_sch (KiCad schematic)
At the start: 16 parts, among them SW2 PTS526_SK15_SMTR2_LFS, SW3 PTS526_SK15_SMTR2_LFS, SW4 PTS526_SK15_SMTR2_LFS, SW5 PTS526_SK15_SMTR2_LFS, SW6 PTS526_SK15_SMTR2_LFS, SW7 PTS526_SK15_SMTR2_LFS, SW8 PTS526_SK15_SMTR2_LFS, SW9 PTS526_SK15_SMTR2_LFS

Commit message: Final version (2026) sent to production
Parts:
- removed SW2, SW3, SW4, SW5, SW6, SW7, SW8, SW9: PTS526_SK15_SMTR2_LFS, footprints:PTS526SK15SMTR2LFS, symbol PTS526_SK15_SMTR2_LFS:PTS526_SK15_SMTR2_LFS
- added SW1, SW2, SW3, SW4, SW5, SW6, SW7, SW8: PTS526_SK15_SMTR2_LFS, footprints:PTS526SK15SMTR2LFS, symbol fabien:PTS526_SK15_SMTR2_LFS
Connections:
- net O_1: now also SW1.1, SW4.1, SW7.1
- net O_2: now also SW2.1, SW5.1, SW8.1
- net O_3: now also SW3.1, SW6.1
- net at D7.2 (A): now also SW5.2
- net at D1.2 (A): now also SW1.2
- net at D8.2 (A): now also SW8.2
- net at D10.2 (A): now also SW6.2
- net at D6.2 (A): now also SW2.2
- net at D3.2 (A): now also SW7.2
- net at D9.2 (A): now also SW3.2
- net at D2.2 (A): now also SW4.2
